Commit message: urdf model spawn+world to base tf+obstacle detection changes

File: model/iris_with_depth_cam_urdf/model.urdf (robot description, URDF)
Before this commit: robot iris_with_depth_cam, 11 links, 10 joints
Links:
- removed link dummy_link
- removed link world
- added link gps_link, mass 0.01
- link cam_link: mass 0.01 -> None
Joints:
- removed joint dummy_to_base
- removed joint world_to_dummy
- added joint iris/gps_joint: type fixed, parent base_link, child gps_link, origin xyz=0      0      0.19492 rpy=0 0 0, axis 0 0 1, limit lower=0.0 upper=0.0 effort=0.0 velocity=0.0
- joint camera_joint: origin xyz=0      0      0 rpy=0 0 0 -> xyz=0      0      0.125 rpy=0 0 0
- joint rotor_0_joint: limit lower=-1e+16 upper=1e+16 effort=0.0 velocity=0.0 -> lower=-1e+16 upper=1e+16 effort=2000.0 velocity=838.0
- joint rotor_1_joint: limit lower=-1e+16 upper=1e+16 effort=0.0 velocity=0.0 -> lower=-1e+16 upper=1e+16 effort=2000.0 velocity=838.0
- joint rotor_2_joint: limit lower=-1e+16 upper=1e+16 effort=0.0 velocity=0.0 -> lower=-1e+16 upper=1e+16 effort=2000.0 velocity=838.0
- joint rotor_3_joint: limit lower=-1e+16 upper=1e+16 effort=0.0 velocity=0.0 -> lower=-1e+16 upper=1e+16 effort=2000.0 velocity=838.0
